Commit message: update deleting generated csv

File: test.urdf (robot description, URDF)
Before this commit: robot pepe, 6 links, 5 joints
Links:
- removed link 12
- removed link 13
- removed link 25
- added link 15, mass 0.4548908082750577; collision cylinder length=0.7644841341148827 radius=0.4352055308828484; visual cylinder length=0.7644841341148827 radius=0.4352055308828484
- added link 19, mass 0.4548908082750577; collision cylinder length=0.7644841341148827 radius=0.4352055308828484; visual cylinder length=0.7644841341148827 radius=0.4352055308828484
- added link 210, mass 0.020112097190324068; collision cylinder length=0.0794222887828453 radius=0.2839112122044005; visual cylinder length=0.0794222887828453 radius=0.2839112122044005
- added link 211, mass 0.020112097190324068; collision cylinder length=0.0794222887828453 radius=0.2839112122044005; visual cylinder length=0.0794222887828453 radius=0.2839112122044005
- added link 212, mass 0.020112097190324068; collision cylinder length=0.0794222887828453 radius=0.2839112122044005; visual cylinder length=0.0794222887828453 radius=0.2839112122044005
- added link 22, mass 0.020112097190324068; collision cylinder length=0.0794222887828453 radius=0.2839112122044005; visual cylinder length=0.0794222887828453 radius=0.2839112122044005
- added link 23, mass 0.020112097190324068; collision cylinder length=0.0794222887828453 radius=0.2839112122044005; visual cylinder length=0.0794222887828453 radius=0.2839112122044005
- added link 26, mass 0.020112097190324068; collision cylinder length=0.0794222887828453 radius=0.2839112122044005; visual cylinder length=0.0794222887828453 radius=0.2839112122044005
- added link 27, mass 0.020112097190324068; collision cylinder length=0.0794222887828453 radius=0.2839112122044005; visual cylinder length=0.0794222887828453 radius=0.2839112122044005
- added link 28, mass 0.020112097190324068; collision cylinder length=0.0794222887828453 radius=0.2839112122044005; visual cylinder length=0.0794222887828453 radius=0.2839112122044005
- link 0: mass 0.005111548388886505 -> 0.9334285853652872; geometry collision cylinder length=1.1562384021383127 radius=0.5069229075824018; visual cylinder length=1.1562384021383127 radius=0.5069229075824018
- link 11: mass 0.8967812290356305 -> 0.4548908082750577; geometry collision cylinder length=0.7644841341148827 radius=0.4352055308828484; visual cylinder length=0.7644841341148827 radius=0.4352055308828484
- link 24: mass 0.9129793571334045 -> 0.020112097190324068; geometry collision cylinder length=0.0794222887828453 radius=0.2839112122044005; visual cylinder length=0.0794222887828453 radius=0.2839112122044005
Joints:
- removed joint 12_to_0
- removed joint 13_to_0
- removed joint 24_to_0
- removed joint 25_to_0
- added joint 15_to_0: type revolute, parent 0, child 15, origin xyz=0.7829853995477848 0.9231142079986676 0.9164696398881665 rpy=6.722454835508084 3.4361420756585797 2.5435158716784105, axis 0 0 1, limit lower=3.1415 upper=-3.1415 effort=1 velocity=1
- added joint 19_to_0: type revolute, parent 0, child 19, origin xyz=0.7829853995477848 0.9231142079986676 0.9164696398881665 rpy=8.963273114010779 3.4361420756585797 2.5435158716784105, axis 0 0 1, limit lower=3.1415 upper=-3.1415 effort=1 velocity=1
- added joint 210_to_19: type revolute, parent 19, child 210, origin xyz=0.14872723056298542 0.10338023596805801 0.9197686401355749 rpy=8.791941490947508 0.48011350943259956 1.8154312825067496, axis 0 0 1, limit lower=3.1415 upper=-3.1415 effort=1 velocity=1
- added joint 211_to_19: type revolute, parent 19, child 211, origin xyz=0.14872723056298542 0.10338023596805801 0.9197686401355749 rpy=13.187912236421262 0.48011350943259956 1.8154312825067496, axis 0 0 1, limit lower=3.1415 upper=-3.1415 effort=1 velocity=1
- added joint 212_to_19: type revolute, parent 19, child 212, origin xyz=0.14872723056298542 0.10338023596805801 0.9197686401355749 rpy=17.583882981895016 0.48011350943259956 1.8154312825067496, axis 0 0 1, limit lower=3.1415 upper=-3.1415 effort=1 velocity=1
- added joint 22_to_11: type revolute, parent 11, child 22, origin xyz=0.14872723056298542 0.10338023596805801 0.9197686401355749 rpy=8.791941490947508 0.48011350943259956 1.8154312825067496, axis 0 0 1, limit lower=3.1415 upper=-3.1415 effort=1 velocity=1
- added joint 23_to_11: type revolute, parent 11, child 23, origin xyz=0.14872723056298542 0.10338023596805801 0.9197686401355749 rpy=13.187912236421262 0.48011350943259956 1.8154312825067496, axis 0 0 1, limit lower=3.1415 upper=-3.1415 effort=1 velocity=1
- added joint 24_to_11: type revolute, parent 11, child 24, origin xyz=0.14872723056298542 0.10338023596805801 0.9197686401355749 rpy=17.583882981895016 0.48011350943259956 1.8154312825067496, axis 0 0 1, limit lower=3.1415 upper=-3.1415 effort=1 velocity=1
- added joint 26_to_15: type revolute, parent 15, child 26, origin xyz=0.14872723056298542 0.10338023596805801 0.9197686401355749 rpy=8.791941490947508 0.48011350943259956 1.8154312825067496, axis 0 0 1, limit lower=3.1415 upper=-3.1415 effort=1 velocity=1
- added joint 27_to_15: type revolute, parent 15, child 27, origin xyz=0.14872723056298542 0.10338023596805801 0.9197686401355749 rpy=13.187912236421262 0.48011350943259956 1.8154312825067496, axis 0 0 1, limit lower=3.1415 upper=-3.1415 effort=1 velocity=1
- added joint 28_to_15: type revolute, parent 15, child 28, origin xyz=0.14872723056298542 0.10338023596805801 0.9197686401355749 rpy=17.583882981895016 0.48011350943259956 1.8154312825067496, axis 0 0 1, limit lower=3.1415 upper=-3.1415 effort=1 velocity=1
- joint 11_to_0: origin xyz=0.44315108729317687 0.5460804203469618 0.9235436492267407 rpy=1.065111308460958 2.3770825431220155 4.447034410361134 -> xyz=0.7829853995477848 0.9231142079986676 0.9164696398881665 rpy=4.481636557005389 3.4361420756585797 2.5435158716784105
